File: PCB_BOARD/ST_prot.kicad_sch (KiCad schematic)
At the start: 28 parts, among them J1 USB_B_Micro, J2 Conn_01x15, J3 Conn_01x15, SW2 SW_Push, U1 XC6206P332MR, U2 STM32F103C8T6, Y1 8MHz

Commit message: Edit footprint and reroute pcb
Parts:
- removed FB1: 100R, Inductor_SMD:L_0805_2012Metric, symbol Device:Ferrite_Bead_Small
- removed R1, R3: 1k5, Resistor_SMD:R_0603_1608Metric, symbol Device:R_Small
- removed U1: XC6206P332MR, Package_TO_SOT_SMD:SOT-23, symbol Regulator_Linear:XC6206PxxxMR
- added C12: 1u, Capacitor_SMD:C_0603_1608Metric, symbol Device:C_Small
- added U3: XC6210B332MR, Package_TO_SOT_SMD:SOT-23-5, symbol Regulator_Linear:XC6210B332MR
- C10, C11, C4, C5, C6, C7, C8, C9: footprint Capacitor_SMD:C_0402_1005Metric -> Capacitor_SMD:C_0603_1608Metric
- SW2: footprint Button_Switch_SMD:SW_Push_SPST_NO_Alps_SKRK -> Button_Switch_SMD:SW_SPST_CK_RS282G05A3
- Y1: footprint Crystal:Crystal_SMD_5032-2Pin_5.0x3.2mm -> Crystal:Crystal_SMD_HC49-SD
Connections:
- net VCC is gone; now on net +5V: C1.1
- net +3.3V: now also U3.5 (VOUT)
- net +5V: now also C12.1, U3.1 (VIN), U3.3 (CE)
- net GND: now also D1.1 (K), D2.1 (K), C12.2, U3.2 (GND)
Other:
- moved on the sheet: C1, C2, D1

Commit message: Finish prototype v1 PCB
Parts:
- removed L1: 27n, Inductor_SMD:L_0402_1005Metric, symbol Device:L_Small
- C1: footprint Capacitor_SMD:C_0603_1608Metric -> Capacitor_SMD:C_0603_1608Metric_Pad1.08x0.95mm_HandSolder
Connections:
- net +3.3VA is gone; now on net +3.3V: C8.1, C9.1, U2.9 (VDDA)
Other:
- note added: "STM32F1 Prototype Board"
- note removed: "STM32F1 Breakout Board"
Changed lines of the file:
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@@
-    (stroke (width 0) (type default))
-  )
-  (wire (pts (xy 231.14 39.37) (xy 234.95 39.37))
     (stroke (width 0) (type default))
   )
@@
     (stroke (width 0) (type default))
   )
-  (wire (pts (xy 240.03 39.37) (xy 243.84 39.37))
+  (wire (pts (xy 231.14 39.37) (xy 243.84 39.37))
     (stroke (width 0) (type default))
   )
@@
     (effects (font (size 2.0066 2.0066) (thickness 0.4013) bold) (justify left bottom))
   )
-  (text "STM32F1 Breakout Board" (at 25.4 25.4 0)
+  (text "STM32F1 Prototype Board" (at 25.4 25.4 0)
     (effects (font (size 5.0038 5.0038) (thickness 1.0008) bold) (justify left bottom))
   )
@@
     )
   )
-  (symbol (lib_id "Device:L_Small") (at 237.49 39.37 90) (unit 1)
-    (in_bom yes) (on_board yes) (dnp no)
-    (property "Reference" "L1" (at 237.49 34.671 90)
-      (effects (font (size 1.27 1.27)))
-    )
-    (property "Value" "27n" (at 237.49 36.9824 90)
-      (effects (font (size 1.27 1.27)))
-    )
-    (property "Footprint" "Inductor_SMD:L_0402_1005Metric" (at 237.49 39.37 0)
-      (effects (font (size 1.27 1.27)) hide)
-    )
-    (property "Datasheet" "~" (at 237.49 39.37 0)
-      (effects (font (size 1.27 1.27)) hide)
-    )
-    (property "LCSC Part #" "C18830" (at 237.49 39.37 0)
+  (symbol (lib_id "Device:C_Small") (at 243.84 43.18 0) (unit 1)
+    (in_bom yes) (on_board yes) (dnp no)
+    (property "Reference" "C8" (at 246.1768 42.0116 0)
+      (effects (font (size 1.27 1.27)) (justify left))
+    )
+    (property "Value" "1u" (at 246.1768 44.323 0)
+      (effects (font (size 1.27 1.27)) (justify left))
+    )
+    (property "Footprint" "Capacitor_SMD:C_0603_1608Metric" (at 243.84 43.18 0)
+      (effects (font (size 1.27 1.27)) hide)
+    )
+    (property "Datasheet" "~" (at 243.84 43.18 0)
+      (effects (font (size 1.27 1.27)) hide)
+    )
+    (property "LCSC Part #" "C52923" (at 243.84 43.18 0)
       (effects (font (size 1.27 1.27)) hide)
     )
@@
       (project "ST_prot"
         (path "/4ba01d44-65dc-426c-acc2-325858297e9f"
-          (reference "L1") (unit 1)
-        )
-      )
-    )
-  )
-  (symbol (lib_id "Device:C_Small") (at 243.84 43.18 0) (unit 1)
-    (in_bom yes) (on_board yes) (dnp no)
-    (property "Reference" "C8" (at 246.1768 42.0116 0)
-      (effects (font (size 1.27 1.27)) (justify left))
-    )
-    (property "Value" "1u" (at 246.1768 44.323 0)
-      (effects (font (size 1.27 1.27)) (justify left))
-    )
-    (property "Footprint" "Capacitor_SMD:C_0603_1608Metric" (at 243.84 43.18 0)
-      (effects (font (size 1.27 1.27)) hide)
-    )
-    (property "Datasheet" "~" (at 243.84 43.18 0)
-      (effects (font (size 1.27 1.27)) hide)
-    )
-    (property "LCSC Part #" "C52923" (at 243.84 43.18 0)
+          (reference "C8") (unit 1)
+        )
+      )
+    )
+  )
+  (symbol (lib_id "Device:C_Small") (at 252.73 43.18 0) (unit 1)
+    (in_bom yes) (on_board yes) (dnp no)
+    (property "Reference" "C9" (at 255.0668 42.0116 0)
+      (effects (font (size 1.27 1.27)) (justify left))
+    )
+    (property "Value" "100n" (at 255.0668 44.323 0)
+      (effects (font (size 1.27 1.27)) (justify left))
+    )
+    (property "Footprint" "Capacitor_SMD:C_0603_1608Metric" (at 252.73 43.18 0)
+      (effects (font (size 1.27 1.27)) hide)
+    )
+    (property "Datasheet" "~" (at 252.73 43.18 0)
+      (effects (font (size 1.27 1.27)) hide)
+    )
+    (property "LCSC Part #" "C1525" (at 252.73 43.18 0)
       (effects (font (size 1.27 1.27)) hide)
     )
@@
       (project "ST_prot"
         (path "/4ba01d44-65dc-426c-acc2-325858297e9f"
-          (reference "C8") (unit 1)
-        )
-      )
-    )
-  )
-  (symbol (lib_id "Device:C_Small") (at 252.73 43.18 0) (unit 1)
-    (in_bom yes) (on_board yes) (dnp no)
-    (property "Reference" "C9" (at 255.0668 42.0116 0)
-      (effects (font (size 1.27 1.27)) (justify left))
-    )
-    (property "Value" "100n" (at 255.0668 44.323 0)
-      (effects (font (size 1.27 1.27)) (justify left))
-    )
-    (property "Footprint" "Capacitor_SMD:C_0603_1608Metric" (at 252.73 43.18 0)
-      (effects (font (size 1.27 1.27)) hide)
-    )
-    (property "Datasheet" "~" (at 252.73 43.18 0)
-      (effects (font (size 1.27 1.27)) hide)
-    )
-    (property "LCSC Part #" "C1525" (at 252.73 43.18 0)
+          (reference "C9") (unit 1)
+        )
+      )
+    )
+  )
+  (symbol (lib_id "power:GND") (at 168.91 48.26 0) (unit 1)
+    (in_bom yes) (on_board yes) (dnp no)
+    (property "Reference" "#PWR019" (at 168.91 54.61 0)
+      (effects (font (size 1.27 1.27)) hide)
+    )
+    (property "Value" "GND" (at 168.91 52.07 0)
+      (effects (font (size 1.27 1.27)))
+    )
+    (property "Footprint" "" (at 168.91 48.26 0)
+      (effects (font (size 1.27 1.27)) hide)
+    )
+    (property "Datasheet" "" (at 168.91 48.26 0)
+      (effects (font (size 1.27 1.27)) hide)
+    )
+    (pin "1")
+    (instances
+      (project "ST_prot"
+        (path "/4ba01d44-65dc-426c-acc2-325858297e9f"
+          (reference "#PWR019") (unit 1)
+        )
+      )
+    )
+  )
+  (symbol (lib_id "Device:C_Small") (at 168.91 43.18 0) (unit 1)
+    (in_bom yes) (on_board yes) (dnp no)
+    (property "Reference" "C3" (at 171.2468 42.0116 0)
+      (effects (font (size 1.27 1.27)) (justify left))
+    )
+    (property "Value" "4u7" (at 171.2468 44.323 0)
+      (effects (font (size 1.27 1.27)) (justify left))
+    )
+    (property "Footprint" "Capacitor_SMD:C_0603_1608Metric" (at 168.91 43.18 0)
+      (effects (font (size 1.27 1.27)) hide)
+    )
+    (property "Datasheet" "~" (at 168.91 43.18 0)
+      (effects (font (size 1.27 1.27)) hide)
+    )
+    (property "LCSC Part #" "C19666" (at 168.91 43.18 0)
       (effects (font (size 1.27 1.27)) hide)
     )
@@
       (project "ST_prot"
         (path "/4ba01d44-65dc-426c-acc2-325858297e9f"
-          (reference "C9") (unit 1)
-        )
-      )
-    )
-  )
-  (symbol (lib_id "power:GND") (at 168.91 48.26 0) (unit 1)
-    (in_bom yes) (on_board yes) (dnp no)
-    (property "Reference" "#PWR019" (at 168.91 54.61 0)
-      (effects (font (size 1.27 1.27)) hide)
-    )
-    (property "Value" "GND" (at 168.91 52.07 0)
-      (effects (font (size 1.27 1.27)))
-    )
-    (property "Footprint" "" (at 168.91 48.26 0)
-      (effects (font (size 1.27 1.27)) hide)
-    )
-    (property "Datasheet" "" (at 168.91 48.26 0)
-      (effects (font (size 1.27 1.27)) hide)
-    )
-    (pin "1")
-    (instances
-      (project "ST_prot"
-        (path "/4ba01d44-65dc-426c-acc2-325858297e9f"
-          (reference "#PWR019") (unit 1)
-        )
-      )
-    )
-  )
-  (symbol (lib_id "Device:C_Small") (at 168.91 43.18 0) (unit 1)
-    (in_bom yes) (on_board yes) (dnp no)
-    (property "Reference" "C3" (at 171.2468 42.0116 0)
-      (effects (font (size 1.27 1.27)) (justify left))
-    )
-    (property "Value" "4u7" (at 171.2468 44.323 0)
-      (effects (font (size 1.27 1.27)) (justify left))
-    )
-    (property "Footprint" "Capacitor_SMD:C_0603_1608Metric" (at 168.91 43.18 0)
-      (effects (font (size 1.27 1.27)) hide)
-    )
-    (property "Datasheet" "~" (at 168.91 43.18 0)
-      (effects (font (size 1.27 1.27)) hide)
-    )
-    (property "LCSC Part #" "C19666" (at 168.91 43.18 0)
-      (effects (font (size 1.27 1.27)) hide)
-    )
-    (pin "1")
-    (pin "2")
-    (instances
-      (project "ST_prot"
-        (path "/4ba01d44-65dc-426c-acc2-325858297e9f"
           (reference "C3") (unit 1)
         )
@@
       (effects (font (size 1.27 1.27)) (justify left))
     )
-    (property "Footprint" "Capacitor_SMD:C_0603_1608Metric" (at 64.77 60.96 0)
-      (effects (font (size 1.27 1.27)) hide)
-    )
+    (property "Footprint" "Capacitor_SMD:C_0603_1608Metric_Pad1.08x0.95mm_HandSolder" (at 64.77 60.96 0)
+      (effects (font (size 1.27 1.27)) hide)
+    )
